Commit message: Almost final simulator. Camera is calibrated and usable. Lidar works just fine as well. The only thing left to do is to auto generate tracks or opponents.

File: src/simulator/selfie-simulator/selfie_description/urdf/macros.xacro (robot description, xacro)
@@ -1,4 +1,4 @@
 <?xml version="1.0"?>
-<robot name="racecar" xmlns:xacro="http://www.ros.org/wiki/xacro">
+<robot name="selfie" xmlns:xacro="http://www.ros.org/wiki/xacro">
 <!-- inertial parameter macros -->
 <xacro:macro name="chassis_inertial_params">
@@ -41,5 +41,5 @@
   <origin xyz="0 0 0" rpy="0 0 0" />
   <geometry>
-    <mesh filename="package://racecar_description/meshes/chassis.STL" />
+    <mesh filename="package://selfie_description/meshes/chassis.STL" />
   </geometry>
 </xacro:macro>
@@ -47,5 +47,5 @@
   <origin xyz="0 0 0" rpy="0 0 0" />
   <geometry>
-    <mesh filename="package://racecar_description/meshes/left_rear_wheel.STL" />
+    <mesh filename="package://selfie_description/meshes/left_rear_wheel.STL" />
   </geometry>
 </xacro:macro>
@@ -53,5 +53,5 @@
   <origin xyz="0 0 0" rpy="0 0 0" />
   <geometry>
-    <mesh filename="package://racecar_description/meshes/right_rear_wheel.STL" />
+    <mesh filename="package://selfie_description/meshes/right_rear_wheel.STL" />
   </geometry>
 </xacro:macro>
@@ -59,5 +59,5 @@
   <origin xyz="0 0 0" rpy="0 0 0" />
   <geometry>
-    <mesh filename="package://racecar_description/meshes/left_front_wheel.STL" />
+    <mesh filename="package://selfie_description/meshes/left_front_wheel.STL" />
   </geometry>
 </xacro:macro>
@@ -65,5 +65,5 @@
   <origin xyz="0 0 0" rpy="0 0 0" />
   <geometry>
-    <mesh filename="package://racecar_description/meshes/right_front_wheel.STL" />
+    <mesh filename="package://selfie_description/meshes/right_front_wheel.STL" />
   </geometry>
 </xacro:macro>
@@ -71,5 +71,5 @@
   <origin xyz="0 0 0" rpy="0 0 0" />
   <geometry>
-    <mesh filename="package://racecar_description/meshes/left_steering_hinge.STL" />
+    <mesh filename="package://selfie_description/meshes/left_steering_hinge.STL" />
   </geometry>
 </xacro:macro>
@@ -77,5 +77,5 @@
   <origin xyz="0 0 0" rpy="0 0 0" />
   <geometry>
-    <mesh filename="package://racecar_description/meshes/right_steering_hinge.STL" />
+    <mesh filename="package://selfie_description/meshes/right_steering_hinge.STL" />
   </geometry>
 </xacro:macro>
@@ -89,5 +89,5 @@
   <origin xyz="0 0 0.0225" rpy="0 0 0" />
   <geometry>
-    <cylinder length="0.045" radius="0.05" />
+    <cylinder length="0.045" radius="0.05" />  <!-- changed from 0.045   -->
   </geometry>
 </xacro:macro>

File: src/simulator/selfie-simulator/selfie_description/urdf/materials.xacro (robot description, xacro)
@@ -1,4 +1,4 @@
 <?xml version="1.0"?>
-<robot name="racecar" xmlns:xacro="http://www.ros.org/wiki/xacro">
+<robot name="selfie" xmlns:xacro="http://www.ros.org/wiki/xacro">
 <material name="black">
   <color rgba="0.0 0.0 0.0 1.0"/>

File: src/simulator/selfie-simulator/selfie_description/urdf/selfie.urdf (robot description, URDF)
Before this commit: robot racecar, 13 links, 12 joints
Links:
- removed link zed_camera_right_link
- link camera_link: geometry collision box size=0.033 0.175 0.030; visual box size=0.033 0.175 0.030
- link chassis: geometry visual mesh filename=package://selfie_description/meshes/chassis.STL
- link laser: geometry collision box size=0.1 0.1 0.1; visual mesh filename=package://selfie_description/meshes/hokuyo.dae
- link left_front_wheel: geometry collision cylinder length=0.045 radius=0.05; visual mesh filename=package://selfie_description/meshes/left_front_wheel.STL
- link left_rear_wheel: geometry collision cylinder length=0.045 radius=0.05; visual mesh filename=package://selfie_description/meshes/left_rear_wheel.STL
- link left_steering_hinge: geometry visual mesh filename=package://selfie_description/meshes/left_steering_hinge.STL
- link right_front_wheel: geometry collision cylinder length=0.045 radius=0.05; visual mesh filename=package://selfie_description/meshes/right_front_wheel.STL
- link right_rear_wheel: geometry collision cylinder length=0.045 radius=0.05; visual mesh filename=package://selfie_description/meshes/right_rear_wheel.STL
- link right_steering_hinge: geometry visual mesh filename=package://selfie_description/meshes/right_steering_hinge.STL
- link zed_camera_link: geometry 
Joints:
- removed joint zed_camera_joint
- removed joint zed_camera_right_joint
- added joint main_camera_joint: type fixed, parent chassis, child camera_link, origin xyz=0.390 0 0.1 rpy=0 30 0, axis 0 0 1
- joint zed_camera_left_joint: child camera_link -> zed_camera_link; parent zed_camera_link -> camera_link

File: src/simulator/selfie-simulator/selfie_description/urdf/selfie_experimental.xacro (robot description, xacro)
@@ -171,54 +171,61 @@
   </joint>
   <!-- zed camera -->
-  <link name="base_camera_link">
+  <link name="zed_camera_link">
     <inertial>
       <mass value="1e-5" />
-      <origin xyz="0 0 0.2" rpy="0 8 0"/>
+      <origin xyz="0 0 0.1" rpy="0 10 0"/>
       <inertia ixx="1e-6" ixy="0" ixz="0" iyy="1e-6" iyz="0" izz="1e-6" />
     </inertial>
     <collision>
-      <origin xyz="0 0 0" rpy="0 5 0"/>
-      <geometry>
-        <box size="0.05 0.04 0.030"/>
-      </geometry>
-    </collision>
-    <visual>
-      <origin xyz="0 0 0" rpy="0 5 0"/>
-      <geometry>
-        <box size="0.05 0.04 0.030"/>
+      <origin xyz="0 0 0" rpy="0 0 0"/>
+      <geometry>
+        <box size="0.033 0.175 0.030"/>
+      </geometry>
+    </collision>
+    <visual>
+      <origin xyz="0 0 0" rpy="0 0 0"/>
+      <geometry>
+        <box size="0.033 0.175 0.030"/>
       </geometry>
       <material name="red"/>
     </visual>
   </link>
-  <joint name="base_camera_joint" type="fixed">
-    <origin xyz="0 0 0.04" rpy="0 0 0"/>
+  <joint name="zed_camera_joint" type="fixed">
+    <origin xyz="0.390 0 0.04" rpy="0 0 0"/>
     <parent link="chassis"/>
-    <child link="base_camera_link"/>
+    <child link="zed_camera_link"/>
     <axis xyz="0 0 1" />
     <!-- <limit lower="0.0" upper="0.0" effort="0.0" velocity="0.0" /> -->
   </joint>
-  <!-- camera lenses -->
+  <!-- zed camera lenses -->
   <!-- It seems these have to have a non-zero mass to have a camera attached? -->
-  <link name="camera_link">
+  <link name="camera_link"><!-- this needs to match the name in zed_wrapper/zed_tf.launch -->
     <inertial>
       <mass value="1e-5" />
-      <origin xyz="0 0 0.4" rpy="0 0.26 0"/>
+      <origin xyz="0 0 0" rpy="0 0 0"/>
       <inertia ixx="1e-6" ixy="0" ixz="0" iyy="1e-6" iyz="0" izz="1e-6" />
     </inertial>
-    <visual>
-      <origin xyz="0 0 0.4" rpy="0 0.26 0"/>
-      <geometry>
-        <box size="0.05 0.02 0.05"/>
-      </geometry>
-      <material name="yellow"/>
-    </visual>
-  </link>
-  <joint name="lens_joint" type="fixed">
-    <origin xyz="0 0 0.4" rpy="0 0.26 0"/>
-    <parent link="base_camera_link"/>
+  </link>
+  <link name="zed_camera_right_link">
+    <inertial>
+      <mass value="1e-5" />
+      <origin xyz="0 0 0" rpy="0 0 0"/>
+      <inertia ixx="1e-6" ixy="0" ixz="0" iyy="1e-6" iyz="0" izz="1e-6" />
+    </inertial>
+  </link>
+  <joint name="zed_camera_left_joint" type="fixed">
+    <origin xyz="0 0.06 0" rpy="0 0 0"/>
+    <parent link="zed_camera_link"/>
     <child link="camera_link"/>
     <axis xyz="0 0 1" />
   </joint>
-<xacro:include filename="$(find selfie_description)/urdf/selfie.gazebo" />
-<xacro:include filename="$(find selfie_description)/urdf/materials.xacro" />
+  <joint name="zed_camera_right_joint" type="fixed">
+    <origin xyz="0 -0.06 0" rpy="0 0 0"/>
+    <parent link="zed_camera_link"/>
+    <child link="zed_camera_right_link"/>
+    <axis xyz="0 0 1" />
+  </joint>
+  <!-- Add the remaining xacros -->
+  <xacro:include filename="$(find selfie_description)/urdf/selfie.gazebo" />
+  <xacro:include filename="$(find selfie_description)/urdf/materials.xacro" />
 </robot>
