Commit message: general structure corrected

File: src/simulator/selfie-simulator/selfie_description/urdf/movable_box.urdf (robot description, URDF)
Before this commit: robot movable_box, 1 links, 0 joints
Links:
- link movable_box_link: geometry collision box size=0.4 0.2 0.2; visual box size=0.4 0.2 0.2
